Commit message: All relevant description changes

File: kassow_kord_description/kr810/urdf/kr810_description_patched_42.urdf.xacro (robot description, xacro)
@@ -33,9 +33,9 @@
       </collision>
   </xacro:macro>
-  <xacro:macro name="visual_and_collision_mesh" params="xyz rpy color mesh_file scale">
+  <xacro:macro name="visual_and_collision_mesh" params="xyz rpy color visual_mesh_file collision_mesh_file scale">
     <visual>
       <origin rpy="${rpy}" xyz="${xyz}" />
       <geometry>
-        <mesh filename="${mesh_file}" scale="${scale}"/>
+        <mesh filename="${visual_mesh_file}" scale="${scale}"/>
       </geometry>
       <material name="">
@@ -46,5 +46,5 @@
       <origin rpy="${rpy}" xyz="${xyz}" />
       <geometry>
-        <mesh filename="${mesh_file}" scale="${scale}"/>
+        <mesh filename="${collision_mesh_file}" scale="${scale}"/>
       </geometry>
     </collision>
@@ -67,5 +67,6 @@
       rpy="0 0 0"
       color="0.2 0.2 0.2 1"
-      mesh_file="package://kassow_kord_description/kr810/meshes/a810/a810_Base.stl"
+      visual_mesh_file="package://kassow_kord_description/kr810/meshes/a810/a810_Base.stl"
+      collision_mesh_file="package://kassow_kord_description/kr810/meshes/a810/a810_Base_collision.stl"
       scale="0.001 0.001 0.001"/>
   </link>
@@ -87,5 +88,6 @@
       rpy="0 0 0"
       color="0.2 0.2 0.2 1"
-      mesh_file="package://kassow_kord_description/kr810/meshes/a810/a810_Link2.stl"
+      visual_mesh_file="package://kassow_kord_description/kr810/meshes/a810/a810_Link2.stl"
+      collision_mesh_file="package://kassow_kord_description/kr810/meshes/a810/a810_Link2_collision.stl"
       scale="0.001 0.001 0.001"/>
   </link>
@@ -122,5 +124,6 @@
       rpy="-${pi/2} 0 -${pi/2}"
       color="0.2 0.2 0.2 1"
-      mesh_file="package://kassow_kord_description/kr810/meshes/a810/a810_Link3.stl"
+      visual_mesh_file="package://kassow_kord_description/kr810/meshes/a810/a810_Link3.stl"
+      collision_mesh_file="package://kassow_kord_description/kr810/meshes/a810/a810_Link3_collision.stl"
       scale="0.001 0.001 0.001"/>
   </link>
@@ -143,5 +146,6 @@
       rpy="${pi/2} 0 -${pi/2}"
       color="0.2 0.2 0.2 1"
-      mesh_file="package://kassow_kord_description/kr810/meshes/a810/a810_Link4.stl"
+      visual_mesh_file="package://kassow_kord_description/kr810/meshes/a810/a810_Link4.stl"
+      collision_mesh_file="package://kassow_kord_description/kr810/meshes/a810/a810_Link4_collision.stl"
       scale="0.001 0.001 0.001"/>
   </link>
@@ -178,5 +182,6 @@
       rpy="-${pi/2} 0 ${pi/2}"
       color="0.2 0.2 0.2 1"
-      mesh_file="package://kassow_kord_description/kr810/meshes/a810/a810_Link5.stl"
+      visual_mesh_file="package://kassow_kord_description/kr810/meshes/a810/a810_Link5.stl"
+      collision_mesh_file="package://kassow_kord_description/kr810/meshes/a810/a810_Link5_collision.stl"
       scale="0.001 0.001 0.001"/>
   </link>
@@ -196,5 +201,6 @@
       rpy="0 0 -${pi/2}"
       color="0.2 0.2 0.2 1"
-      mesh_file="package://kassow_kord_description/kr810/meshes/a810/a810_Link6.stl"
+      visual_mesh_file="package://kassow_kord_description/kr810/meshes/a810/a810_Link6.stl"
+      collision_mesh_file="package://kassow_kord_description/kr810/meshes/a810/a810_Link6_collision.stl"
       scale="0.001 0.001 0.001"/>
   </link>
@@ -231,5 +237,6 @@
       rpy="0 0 0"
       color="0.2 0.2 0.2 1"
-      mesh_file="package://kassow_kord_description/kr810/meshes/a810/a810_Link7.stl"
+      visual_mesh_file="package://kassow_kord_description/kr810/meshes/a810/a810_Link7.stl"
+      collision_mesh_file="package://kassow_kord_description/kr810/meshes/a810/a810_Link7_collision.stl"
       scale="0.001 0.001 0.001"/>
   </link>
@@ -251,5 +258,6 @@
       rpy="0 0 0"
       color="0.8 0.8 0.8 1"
-      mesh_file="package://kassow_kord_description/kr810/meshes/a810/a810_ToolIO.stl"
+      visual_mesh_file="package://kassow_kord_description/kr810/meshes/a810/a810_ToolIO.stl"
+      collision_mesh_file="package://kassow_kord_description/kr810/meshes/a810/a810_ToolIO_collision.stl"
       scale="0.001 0.001 0.001"/>
   </link>
@@ -260,85 +268,131 @@
     <child link="${prefix}_base"/>
   </joint>
+  <xacro:property name="joint0_xoffset" value="${ 0 }" />
+  <xacro:property name="joint0_yoffset" value="${ 0 }" />
+  <xacro:property name="joint0_zoffset" value="${ 0.03493 }" />
+  <xacro:property name="joint0_roll" value="${ 0 }" />
+  <xacro:property name="joint0_pitch" value="${ 0 }" />
+  <xacro:property name="joint0_yaw" value="${ 0 }" />
   <joint name="${prefix}_joint_1" type="revolute">
     <parent link="${prefix}_base"/>
     <child link="${prefix}_link1"/>
-    <origin rpy="0 0 0" xyz="0 0 ${base_inner_height + base_outer_height}"/>
+    <origin rpy="${joint0_roll} ${joint0_pitch} ${joint0_yaw}" xyz="${joint0_xoffset} ${joint0_yoffset} ${joint0_zoffset}"/>
     <axis xyz="0 0 1"/>
     <dynamics damping="${joints_damping}"/>
     <limit effort="60" velocity="${radians(225)}" lower="${-2*pi}" upper="${2*pi}"/>
   </joint>
-  <xacro:property name="joint1_xoffset"  value="${  50.0 * scale}" />
-  <xacro:property name="joint1_yoffset"  value="${   0.0 * scale}" />
-  <xacro:property name="joint1_zoffset"  value="${ 308.7 * scale - 35 * scale}" />
+  <xacro:property name="joint1_xoffset"  value="${ 0.04949767397 }" />
+  <xacro:property name="joint1_yoffset"  value="${ 0 }" />
+  <xacro:property name="joint1_zoffset"  value="${ 0.27322246 }" />
+  <xacro:property name="joint1_roll" value="${ 0.0003147125244 }" />
+  <xacro:property name="joint1_pitch" value="${ 0.0007407422742 }" />
+  <xacro:property name="joint1_yaw" value="${ 2.331208787e-07 }" />
   <joint name="${prefix}_joint_2" type="revolute">
     <parent link="${prefix}_link1"/>
     <child link="${prefix}_linkJ2"/>
-    <origin rpy="0 0 0" xyz="${joint1_xoffset} ${joint1_yoffset} ${joint1_zoffset}"/>
+    <origin rpy="${joint1_roll} ${joint1_pitch} ${joint1_yaw}" xyz="${joint1_xoffset} ${joint1_yoffset} ${joint1_zoffset}"/>
     <axis xyz="0 1 0"/>
     <dynamics damping="${joints_damping}"/>
     <limit effort="60" velocity="${radians(225)}" lower="-${radians(70.0)}" upper="${pi}"/>
   </joint>
-  <xacro:property name="jointPL2_xoffset"  value="${  -50.0 * scale}" />
-  <xacro:property name="jointPL2_yoffset"  value="${  -85.7 * scale}" />
+  <xacro:property name="jointPL2_xoffset"  value="${ -0.05048137719 }" />
+  <xacro:property name="jointPL2_yoffset"  value="${ -0.08545515779 }" />
+  <xacro:property name="jointPL2_zoffset" value="${ 0 }" />
+  <xacro:property name="jointPL2_roll" value="${ -5.273707211e-05 }" />
+  <xacro:property name="jointPL2_pitch" value="${ -3.208353892e-08 }" />
+  <xacro:property name="jointPL2_yaw" value="${ -0.0006083678446 }" />
   <joint name="${prefix}_jointPL2" type="fixed">
     <parent link="${prefix}_linkJ2"/>
     <child link="${prefix}_link2"/>
-    <origin rpy="0 0 0" xyz="${jointPL2_xoffset} ${jointPL2_yoffset} 0"/>
-  </joint>
+    <origin rpy="${jointPL2_roll} ${jointPL2_pitch} ${jointPL2_yaw}" xyz="${jointPL2_xoffset} ${jointPL2_yoffset} ${jointPL2_zoffset}"/>
+  </joint>
+  <xacro:property name="joint2_xoffset" value="${ 0 }" />
+  <xacro:property name="joint2_yoffset" value="${ 0 }" />
+  <xacro:property name="joint2_zoffset" value="${ 0.2790408 }" />
+  <xacro:property name="joint2_roll" value="${ 0 }" />
+  <xacro:property name="joint2_pitch" value="${ 0 }" />
+  <xacro:property name="joint2_yaw" value="${ 0 }" />
   <joint name="${prefix}_joint_3" type="revolute">
     <parent link="${prefix}_link2"/>
     <child link="${prefix}_link3"/>
-    <origin rpy="0 0 0" xyz="0 0 ${link2_length}"/>
+    <origin rpy="${joint2_roll} ${joint2_pitch} ${joint2_yaw}" xyz="${joint2_xoffset} ${joint2_yoffset} ${joint2_zoffset}"/>
     <axis xyz="0 0 1"/>
     <dynamics damping="${joints_damping}"/>
     <limit effort="40" velocity="${radians(225)}" lower="${-2*pi}" upper="${2*pi}"/>
   </joint>
-  <xacro:property name="joint3_xoffset"  value="${ 40.0 * scale}" />
-  <xacro:property name="joint3_yoffset"  value="${ 0.0 * scale}" />
-  <xacro:property name="joint3_zoffset"  value="${ 142.9 * scale}" />
+  <xacro:property name="joint3_xoffset"  value="${ 0.03998057476 }" />
+  <xacro:property name="joint3_yoffset"  value="${ 0 }" />
+  <xacro:property name="joint3_zoffset"  value="${ 0.1375700579 }" />
+  <xacro:property name="joint3_roll" value="${ 0.0008507333696 }" />
+  <xacro:property name="joint3_pitch" value="${ -0.004532946496 }" />
+  <xacro:property name="joint3_yaw" value="${ -3.856329777e-06 }" />
   <joint name="${prefix}_joint_4" type="revolute">
     <parent link="${prefix}_link3"/>
     <child link="${prefix}_linkJ4"/>
-    <origin rpy="0 0 0" xyz="${joint3_xoffset} ${joint3_yoffset} ${joint3_zoffset}"/>
+    <origin rpy="${joint3_roll} ${joint3_pitch} ${joint3_yaw}" xyz="${joint3_xoffset} ${joint3_yoffset} ${joint3_zoffset}"/>
     <axis xyz="0 1 0"/>
     <dynamics damping="${joints_damping}"/>
     <limit effort="40" velocity="${radians(225)}" lower="-${radians(70.0)}" upper="${pi}"/>
   </joint>
-  <xacro:property name="jointPL4_xoffset"  value="${ -40.0 * scale}" />
-  <xacro:property name="jointPL4_yoffset"  value="${ 84.05 * scale}" />
-  <xacro:property name="jointPL4_zoffset"  value="${ 0.0 * scale}" />
+  <xacro:property name="jointPL4_xoffset"  value="${ -0.0396161075 }" />
+  <xacro:property name="jointPL4_yoffset"  value="${ 0.08376852634 }" />
+  <xacro:property name="jointPL4_zoffset"  value="${ 0 }" />
+  <xacro:property name="jointPL4_roll" value="${ 2.963095903e-05 }" />
+  <xacro:property name="jointPL4_pitch" value="${ 9.531149608e-08 }" />
+  <xacro:property name="jointPL4_yaw" value="${ -0.003216618671 }" />
   <joint name="${prefix}_jointPL4" type="fixed">
     <parent link="${prefix}_linkJ4"/>
     <child link="${prefix}_link4"/>
-    <origin rpy="0 0 0" xyz="${jointPL4_xoffset} ${jointPL4_yoffset} ${jointPL4_zoffset}"/>
-  </joint>
+    <origin rpy="${jointPL4_roll} ${jointPL4_pitch} ${jointPL4_yaw}" xyz="${jointPL4_xoffset} ${jointPL4_yoffset} ${jointPL4_zoffset}"/>
+  </joint>
+  <xacro:property name="joint4_xoffset" value="${ 0 }" />
+  <xacro:property name="joint4_yoffset" value="${ 0 }" />
+  <xacro:property name="joint4_zoffset" value="${ 0.273452 }" />
+  <xacro:property name="joint4_roll" value="${ 0 }" />
+  <xacro:property name="joint4_pitch" value="${ 0 }" />
+  <xacro:property name="joint4_yaw" value="${ 0 }" />
   <joint name="${prefix}_joint_5" type="revolute">
     <parent link="${prefix}_link4"/>
     <child link="${prefix}_link5"/>
-    <origin rpy="0 0 0" xyz="0 0 ${link4_length}"/>
+    <origin rpy="${joint4_roll} ${joint4_pitch} ${joint4_yaw}" xyz="${joint4_xoffset} ${joint4_yoffset} ${joint4_zoffset}"/>
     <axis xyz="0 0 1"/>
     <dynamics damping="${joints_damping}"/>
     <limit effort="20" velocity="${radians(225)}" lower="${-2*pi}" upper="${2*pi}"/>
   </joint>
-  <xacro:property name="joint5_zoffset"  value="${ 103.5 * scale}" />
+  <xacro:property name="joint5_zoffset"  value="${ 0.1003510349 }" />
+  <xacro:property name="joint5_xoffset" value="${ -5.850020796e-05 }" />
+  <xacro:property name="joint5_yoffset" value="${ 0 }" />
+  <xacro:property name="joint5_roll" value="${ 0.0004277043045 }" />
+  <xacro:property name="joint5_pitch" value="${ 0.001085242157 }" />
+  <xacro:property name="joint5_yaw" value="${ 4.641627703e-07 }" />
   <joint name="${prefix}_joint_6" type="revolute">
     <parent link="${prefix}_link5"/>
     <child link="${prefix}_linkJ6"/>
-    <origin rpy="0 0 0" xyz="0 0 ${joint5_zoffset}"/>
+    <origin rpy="${joint5_roll} ${joint5_pitch} ${joint5_yaw}" xyz="${joint5_xoffset} ${joint5_yoffset} ${joint5_zoffset}"/>
     <axis xyz="0 1 0"/>
     <dynamics damping="${joints_damping}"/>
     <limit effort="20" velocity="${radians(225)}" lower="${-2*pi}" upper="${2*pi}"/>
   </joint>
-  <xacro:property name="jointPL6_yoffset"  value="${ 111.0 * scale}" />
+  <xacro:property name="jointPL6_yoffset"  value="${ 0.1108804748 }" />
+  <xacro:property name="jointPL6_xoffset" value="${ 1.849439368e-05 }" />
+  <xacro:property name="jointPL6_zoffset" value="${ 0 }" />
+  <xacro:property name="jointPL6_roll" value="${ 0.0002416074276 }" />
+  <xacro:property name="jointPL6_pitch" value="${ 0 }" />
+  <xacro:property name="jointPL6_yaw" value="${ 0 }" />
   <joint name="${prefix}_jointPL6" type="fixed">
     <parent link="${prefix}_linkJ6"/>
     <child link="${prefix}_link6"/>
-    <origin rpy="0 0 0" xyz="0 ${jointPL6_yoffset} 0"/>
-  </joint>
-  <xacro:property name="joint6_zoffset"  value="${ 108.0 * scale}" />
+    <origin rpy="${jointPL6_roll} ${jointPL6_pitch} ${jointPL6_yaw}" xyz="${jointPL6_xoffset} ${jointPL6_yoffset} ${jointPL6_zoffset}"/>
+  </joint>
+  <xacro:property name="joint6_zoffset"  value="${ 0.107784 }" />
+  <xacro:property name="joint6_xoffset" value="${ 0 }" />
+  <xacro:property name="joint6_yoffset" value="${ 0 }" />
+  <xacro:property name="joint6_roll" value="${ 0 }" />
+  <xacro:property name="joint6_pitch" value="${ 0 }" />
+  <xacro:property name="joint6_yaw" value="${ 0 }" />
   <joint name="${prefix}_joint_7" type="revolute">
     <parent link="${prefix}_link6"/>
     <child link="${prefix}_end_effector"/>
-    <origin rpy="0 0 0" xyz="0 0 ${joint6_zoffset}"/>
+    <origin rpy="${joint6_roll} ${joint6_pitch} ${joint6_yaw}" xyz="${joint6_xoffset} ${joint6_yoffset} ${joint6_zoffset}"/>
     <axis xyz="0 0 1"/>
     <dynamics damping="${joints_damping}"/>
