Commit message: URDF and SRDF first pass

File: kassow_kord_bringup/srdf/kassow_kord.srdf.xacro (robot description, xacro)
@@ -2,5 +2,11 @@
 <robot name="kassow_kord" xmlns:xacro="http://wiki.ros.org/xacro">
     <xacro:arg name="prefix" default=""/>
+    <xacro:arg name="hand_type" default="none"/>
+    <xacro:arg name="hand_srdf_file" default=""/>
     <xacro:include filename="$(find kassow_kord_bringup)/srdf/kassow_kord_macro.srdf.xacro"/>
-    <xacro:kassow_kord_srdf prefix="$(arg prefix)"/>
+    <xacro:kassow_kord_srdf
+      prefix="$(arg prefix)"
+      hand_type="$(arg hand_type)"
+      hand_srdf_file="$(arg hand_srdf_file)"
+    />
 </robot>

File: kassow_kord_bringup/srdf/kassow_kord_macro.srdf.xacro (robot description, xacro)
@@ -1,8 +1,15 @@
 <?xml version="1.0" encoding="UTF-8"?>
 <robot name="kassow_kord" xmlns:xacro="http://wiki.ros.org/xacro">
-  <xacro:macro name="kassow_kord_srdf" params="prefix tip_link='end_effector'">
-    <group name="${prefix}_manipulator">
+  <xacro:macro name="kassow_kord_srdf" params="prefix hand_type hand_srdf_file tip_link='end_effector'">
+    <xacro:if value="${hand_type == 'none'}">
+      <group name="${prefix}_manipulator">
         <chain base_link="${prefix}_base" tip_link="${prefix}_${tip_link}"/>
-    </group>
+      </group>
+    </xacro:if>
+    <xacro:unless value="${hand_type == 'none'}">
+      <group name="${prefix}_manipulator">
+        <chain base_link="${prefix}_base" tip_link="${prefix}_grasp"/>
+      </group>
+    </xacro:unless>
     <disable_collisions link1="${prefix}_base" link2="${prefix}_link1" reason="Adjacent" />
     <disable_collisions link1="${prefix}_link1" link2="${prefix}_linkJ2" reason="Adjacent" />
@@ -11,4 +18,5 @@
     <disable_collisions link1="${prefix}_link2" link2="${prefix}_link3" reason="Adjacent" />
     <disable_collisions link1="${prefix}_link3" link2="${prefix}_linkJ4" reason="Adjacent" />
+    <disable_collisions link1="${prefix}_link3" link2="${prefix}_link4" reason="Adjacent" />  <!-- patched -->
     <disable_collisions link1="${prefix}_linkJ4" link2="${prefix}_link4" reason="Adjacent" />
     <disable_collisions link1="${prefix}_link4" link2="${prefix}_link5" reason="Adjacent" />
@@ -17,4 +25,9 @@
     <disable_collisions link1="${prefix}_linkJ6" link2="${prefix}_link6" reason="Adjacent" />
     <disable_collisions link1="${prefix}_link6" link2="${prefix}_end_effector" reason="Adjacent" />
+    <xacro:unless value="${hand_type == 'none'}">
+      <disable_collisions link1="${prefix}_end_effector" link2="${prefix}_hand_link" reason="Adjacent"/>
+      <xacro:include filename="$(arg hand_srdf_file)"/>
+      <xacro:hand_collisions_srdf prefix="${prefix}"/>
+    </xacro:unless>
   </xacro:macro>
 </robot>

File: kassow_kord_bringup/urdf/kassow_kord.urdf.xacro (robot description, xacro)
@@ -3,15 +3,38 @@
   <xacro:arg name="prefix" default="kassow"/>
   <xacro:arg name="use_mock_hardware" default="true"/>
-  <xacro:arg name="ip_address" default="10.23.23.238"/>
-  <xacro:arg name="port" default="28283"/>
+  <xacro:arg name="ip_address" default="192.168.33.2"/>
+  <xacro:arg name="port" default="7582"/>
   <xacro:arg name="session_id" default="1"/>
-  <xacro:include filename="$(find kassow_kord_bringup)/urdf/common/inertials.xacro" />
-  <xacro:include filename="$(find kassow_kord_bringup)/urdf/common/materials.xacro" />
-  <xacro:include filename="$(find kassow_kord_description)/kr810/urdf/kr810_description.urdf.xacro"/>
+  <xacro:arg name="hand_type" default="none"/>
+  <xacro:arg name="robot_serial_number" default="42"/>
+  <xacro:arg name="nominal" default="false"/>
+  <!-- Convert arg -> xacro property so it can be used inside ${...} -->
+  <xacro:property name="hand_type" value="$(arg hand_type)"/>
+  <xacro:property name="robot_serial_number" value="$(arg robot_serial_number)"/>
+  <xacro:property name="nominal" value="$(arg nominal)"/>
+  <xacro:include filename="$(find kassow_kord_bringup)/urdf/common/inertials.xacro"/>
+  <xacro:include filename="$(find kassow_kord_bringup)/urdf/common/materials.xacro"/>
+  <!-- KR810 description selection -->
+  <xacro:if value="${nominal}">
+    <xacro:include filename="$(find kassow_kord_description)/kr810/urdf/kr810_description_nominal.urdf.xacro"/>
+  </xacro:if>
+  <xacro:if value="${not nominal}">
+    <xacro:include filename="$(find kassow_kord_description)/kr810/urdf/kr810_description_patched_${robot_serial_number}.urdf.xacro"/>
+  </xacro:if>
   <xacro:include filename="$(find kassow_kord_bringup)/urdf/kassow_kord.ros2_control.xacro"/>
+  <!-- Hand include -->
+  <xacro:include filename="$(find futur_hand_description)/hands/hand_${hand_type}/urdf/hand_${hand_type}.urdf.xacro"/>
+  <!-- Tree -->
+  <!-- World link -->
   <link name="world"/>
   <xacro:kr810_description prefix="$(arg prefix)" parent="world">
-    <origin xyz="0 0 0" rpy="0 0 0"/>
+    <origin xyz="0 0 0" rpy="0 0 0.785398"/>
   </xacro:kr810_description>
+  <xacro:if value="${hand_type != 'none'}">
+    <xacro:hand_description
+      parent_link="$(arg prefix)_end_effector"
+      prefix="$(arg prefix)"
+    />
+  </xacro:if>
   <xacro:kassow_kord_ros2_control
     name="$(arg prefix)"
